Commit message: move down lidar

File: turtlebot2n_description/urdf/sensors/rplidar.urdf.xacro (robot description, xacro)
@@ -5,5 +5,5 @@
     <joint name="laser_joint" type="fixed">
       <axis xyz="0 1 0" /> <!-- this joint rotates around y axis, defined in the dae file -->
-      <origin xyz="0 0 0.4" rpy="0 0 ${M_PI}" />
+      <origin xyz="0 0 0.19" rpy="0 0 ${M_PI}" />
       <parent link="${parent}" />
       <child link="laser" />
